Commit message: six wheels

File: robot.xacro (robot description, xacro)
@@ -3,7 +3,7 @@
 <!-- sve merne jedinice su u metrima, kilogramima itd... -->
 <xacro:property name="body_link_x_dim" value="1"/>
-<xacro:property name="body_link_y_dim" value="0.7"/>
-<xacro:property name="body_link_z_dim" value="0.05"/>
-<xacro:property name="wheel_link_radius" value="0.3"/>
+<xacro:property name="body_link_y_dim" value="0.6"/>
+<xacro:property name="body_link_z_dim" value="0.3"/>
+<xacro:property name="wheel_link_radius" value="0.15"/>
 <xacro:property name="wheel_link_length" value="0.1"/>
 <xacro:property name="wheel_link_z_location" value="-0.1"/>
@@ -18,11 +18,12 @@
 <xacro:macro name="inertia_wheel">
 	<inertial>
-		<origin rpy="0 0 0" xyz="0 0 0"/>
-		<mass value="${wheel_mass}"/>
-		<inertia ixx="${I_wheel}" ixy="0" ixz="0" iyy="${I_wheel}" iyz="0" izz="${I_wheel}"/>
+	<origin rpy="0 0 0" xyz="0 0 0"/>
+	<mass value="${wheel_mass}"/>
+	<inertia ixx="${I_wheel}" ixy="0" ixz="0" iyy="${I_wheel}" iyz="0" izz="${I_wheel}"/>
 	</inertial>
 </xacro:macro>
 <xacro:include filename="$(find mobile_robot)/model/robot.gazebo"/>
-<link name="dummy"/>
+<link name="dummy">
+</link>
 <joint name="dummy_joint" type="fixed">
 	<parent link="dummy"/>
@@ -30,28 +31,27 @@
 </joint>
 <!--############################################################### -->
-<link name="body_link">
-	<visual>
-		<geometry>
-			<box size="${body_link_x_dim} ${body_link_y_dim} ${body_link_z_dim}"/>
-		</geometry>
-		<origin rpy="0 0 0" xyz="0 0 0"/>
-	</visual>
-	<collision>
-		<geometry>
-			<box size="${body_link_x_dim} ${body_link_y_dim} ${body_link_z_dim}"/>
-		</geometry>
-		<origin rpy="0 0 0" xyz="0 0 0"/>
-	</collision>
-	<inertial>
-		<origin rpy="0 0 0" xyz="0 0 0"/>
-		<mass value="${body_mass}"/>
-		<inertia
-			ixx="${(1.0/12.0)*body_mass*(body_link_y_dim*body_link_y_dim+body_link_z_dim*body_link_z_dim)}"
-			ixy="0"
-			ixz="0"
-			iyy="${(1/12)*body_mass*(body_link_x_dim*body_link_x_dim+body_link_z_dim*body_link_z_dim)}"
-			iyz="0"
-			izz="${(1/12)*body_mass*(body_link_y_dim*body_link_y_dim+body_link_x_dim*body_link_x_dim)}"/>
-	</inertial>
+ <link name="body_link">
+        <visual>
+	    <geometry>
+		<box size="${body_link_x_dim} ${body_link_y_dim} ${body_link_z_dim}"/>
+	    </geometry>
+	    <origin rpy="0 0 0" xyz="0 0 0"/>
+	</visual>
+	<collision>
+	    <geometry>
+		<box size="${body_link_x_dim} ${body_link_y_dim} ${body_link_z_dim}"/>
+	    </geometry>
+	    <origin rpy="0 0 0" xyz="0 0 0"/>
+	</collision>
+        <inertial>
+            <origin rpy="0 0 0" xyz="0 0 0"/>
+            <mass value="${body_mass}"/>
+            <inertia ixx="${(1.0/12.0)*body_mass*(body_link_y_dim*body_link_y_dim+body_link_z_dim*body_link_z_dim)}"
+            ixy="0"
+            ixz="0"
+            iyy="${(1/12)*body_mass*(body_link_x_dim*body_link_x_dim+body_link_z_dim*body_link_z_dim)}"
+            iyz="0"
+            izz="${(1/12)*body_mass*(body_link_y_dim*body_link_y_dim+body_link_x_dim*body_link_x_dim)}"/>
+        </inertial>
 </link>
 <!--############################################################ -->
@@ -59,101 +59,100 @@
 	<parent link="body_link"/>
 	<child link="wheel1_link"/>
-	<origin xyz="-1.0 -0.4 -0.5" rpy="0 0 0" />
-	<axis xyz="0 1 0"/>
-	<limit effort="1000" velocity="1000"/>
-	<dynamics damping="1.0" friction="1.0"/>
-</joint>
-<link name="wheel1_link">
-	<visual>
-		<origin rpy="1.570795 0 0" xyz="0 0 0"/>
-		<geometry>
-			<cylinder length="${wheel_link_length}" radius="${wheel_link_radius}"/>
-		</geometry>
-	</visual>
-	<collision>
-		<origin rpy="1.570795 0 0" xyz="0 0 0"/>
-		<geometry>
-			<cylinder length="${wheel_link_length}" radius="${wheel_link_radius}"/>
-		</geometry>
-	</collision>
-	<xacro:inertia_wheel />
-</link>
-<!-- Front Right Wheel -->
+	<origin xyz="${-body_link_x_dim/2+1.2*wheel_link_radius} ${-body_link_y_dim/2-wheel_link_length/2} ${wheel_link_z_location}" rpy="0 0 0" />
+	<axis xyz="0 1 0"/>
+	<limit effort="1000" velocity="1000"/>
+	<dynamics damping="1.0" friction="1.0"/>
+</joint>
+ <link name="wheel1_link">
+        <visual>
+	    <origin rpy="1.570795 0 0" xyz="0 0 0"/>
+	    <geometry>
+	    <cylinder length="${wheel_link_length}" radius="${wheel_link_radius}"/>
+	    </geometry>
+	</visual>
+	<collision>
+	    <origin rpy="1.570795 0 0" xyz="0 0 0"/>
+	    <geometry>
+	    <cylinder length="${wheel_link_length}" radius="${wheel_link_radius}"/>
+	    </geometry>
+	</collision>
+        <xacro:inertia_wheel />
+</link>
+<!--########################################################## -->
 <joint name="wheel2_joint" type="continuous">
 	<parent link="body_link"/>
 	<child link="wheel2_link"/>
-	<origin xyz="-1.0 0.4 -0.5" rpy="0 0 0"/>
-	<axis xyz="0 1 0"/>
-	<limit effort="1000" velocity="1000"/>
-	<dynamics damping="1.0" friction="1.0"/>
-</joint>
-<link name="wheel2_link">
-	<visual>
-		<origin rpy="1.570795 0 0" xyz="0 0 0"/>
-		<geometry>
-			<cylinder length="${wheel_link_length}" radius="${wheel_link_radius}"/>
-		</geometry>
-	</visual>
-	<collision>
-		<origin rpy="1.570795 0 0" xyz="0 0 0"/>
-		<geometry>
-			<cylinder length="${wheel_link_length}" radius="${wheel_link_radius}"/>
-		</geometry>
-	</collision>
-	<xacro:inertia_wheel />
-</link>
-<!-- Middle Left Wheel -->
+	<origin xyz="${-body_link_x_dim/2+1.2*wheel_link_radius} ${body_link_y_dim/2+wheel_link_length/2} ${wheel_link_z_location}" rpy="0 0 0"/>
+	<axis xyz="0 1 0"/>
+	<limit effort="1000" velocity="1000"/>
+	<dynamics damping="1.0" friction="1.0"/>
+</joint>
+ <link name="wheel2_link">
+        <visual>
+	    <origin rpy="1.570795 0 0" xyz="0 0 0"/>
+	    <geometry>
+	    <cylinder length="${wheel_link_length}" radius="${wheel_link_radius}"/>
+	    </geometry>
+	</visual>
+	<collision>
+	    <origin rpy="1.570795 0 0" xyz="0 0 0"/>
+	    <geometry>
+	    <cylinder length="${wheel_link_length}" radius="${wheel_link_radius}"/>
+	    </geometry>
+	</collision>
+        <xacro:inertia_wheel />
+</link>
+<!--######################################################### -->
 <joint name="wheel3_joint" type="continuous">
 	<parent link="body_link"/>
 	<child link="wheel3_link"/>
-	<origin xyz="0.0 -0.4 -0.5" rpy="0 0 0"/>
-	<axis xyz="0 1 0"/>
-	<limit effort="1000" velocity="1000"/>
-	<dynamics damping="1.0" friction="1.0"/>
-</joint>
-<link name="wheel3_link">
-	<visual>
-		<origin rpy="1.570795 0 0" xyz="0 0 0"/>
-		<geometry>
-			<cylinder length="${wheel_link_length}" radius="${wheel_link_radius}"/>
-		</geometry>
-	</visual>
-	<collision>
-		<origin rpy="1.570795 0 0" xyz="0 0 0"/>
-		<geometry>
-			<cylinder length="${wheel_link_length}" radius="${wheel_link_radius}"/>
-		</geometry>
-	</collision>
-	<xacro:inertia_wheel />
-</link>
-<!-- Middle Right Wheel -->
+	<origin xyz="${body_link_x_dim/2-1.2*wheel_link_radius} ${-body_link_y_dim/2-wheel_link_length/2} ${wheel_link_z_location}" rpy="0 0 0"/>
+	<axis xyz="0 1 0"/>
+	<limit effort="1000" velocity="1000"/>
+	<dynamics damping="1.0" friction="1.0"/>
+</joint>
+ <link name="wheel3_link">
+        <visual>
+	    <origin rpy="1.570795 0 0" xyz="0 0 0"/>
+	    <geometry>
+	    <cylinder length="${wheel_link_length}" radius="${wheel_link_radius}"/>
+	    </geometry>
+	</visual>
+	<collision>
+	    <origin rpy="1.570795 0 0" xyz="0 0 0"/>
+	    <geometry>
+	    <cylinder length="${wheel_link_length}" radius="${wheel_link_radius}"/>
+	    </geometry>
+	</collision>
+        <xacro:inertia_wheel />
+</link>
+<!--######################################################### -->
 <joint name="wheel4_joint" type="continuous">
 	<parent link="body_link"/>
 	<child link="wheel4_link"/>
-	<origin xyz="0.0 0.4 -0.5" rpy="0 0 0"/>
-	<axis xyz="0 1 0"/>
-	<limit effort="1000" velocity="1000"/>
-	<dynamics damping="1.0" friction="1.0"/>
-</joint>
-<link name="wheel4_link">
-	<visual>
-		<origin rpy="1.570795 0 0" xyz="0 0 0"/>
-		<geometry>
-			<cylinder length="${wheel_link_length}" radius="${wheel_link_radius}"/>
-		</geometry>
-	</visual>
-	<collision>
-		<origin rpy="1.570795 0 0" xyz="0 0 0"/>
-		<geometry>
-			<cylinder length="${wheel_link_length}" radius="${wheel_link_radius}"/>
-		</geometry>
-	</collision>
-	<xacro:inertia_wheel />
-</link>
-<!-- Rear Left Wheel -->
+	<origin xyz="${body_link_x_dim/2-1.2*wheel_link_radius} ${body_link_y_dim/2+wheel_link_length/2} ${wheel_link_z_location}" rpy="0 0 0"/>
+	<axis xyz="0 1 0"/>
+	<limit effort="1000" velocity="1000"/>
+	<dynamics damping="1.0" friction="1.0"/>
+</joint>
+ <link name="wheel4_link">
+        <visual>
+	    <origin rpy="1.570795 0 0" xyz="0 0 0"/>
+	    <geometry>
+	    <cylinder length="${wheel_link_length}" radius="${wheel_link_radius}"/>
+	    </geometry>
+	</visual>
+	<collision>
+	    <origin rpy="1.570795 0 0" xyz="0 0 0"/>
+	    <geometry>
+	    <cylinder length="${wheel_link_length}" radius="${wheel_link_radius}"/>
+	    </geometry>
+	</collision>
+        <xacro:inertia_wheel />
+</link>
 <joint name="wheel5_joint" type="continuous">
 	<parent link="body_link"/>
 	<child link="wheel5_link"/>
-	<origin xyz="1.0 -0.4 -0.5" rpy="0 0 0"/>
+	<origin xyz="0 ${-body_link_y_dim/2-wheel_link_length/2} ${wheel_link_z_location}" rpy="0 0 0"/>
 	<axis xyz="0 1 0"/>
 	<limit effort="1000" velocity="1000"/>
@@ -161,23 +160,23 @@
 </joint>
 <link name="wheel5_link">
-	<visual>
-		<origin rpy="1.570795 0 0" xyz="0 0 0"/>
-		<geometry>
-			<cylinder length="${wheel_link_length}" radius="${wheel_link_radius}"/>
-		</geometry>
-	</visual>
-	<collision>
-		<origin rpy="1.570795 0 0" xyz="0 0 0"/>
-		<geometry>
-			<cylinder length="${wheel_link_length}" radius="${wheel_link_radius}"/>
-		</geometry>
-	</collision>
-	<xacro:inertia_wheel />
-</link>
-<!-- Rear Right Wheel -->
+    <visual>
+	    <origin rpy="1.570795 0 0" xyz="0 0 0"/>
+	    <geometry>
+	        <cylinder length="${wheel_link_length}" radius="${wheel_link_radius}"/>
+	    </geometry>
+	</visual>
+	<collision>
+	    <origin rpy="1.570795 0 0" xyz="0 0 0"/>
+	    <geometry>
+	        <cylinder length="${wheel_link_length}" radius="${wheel_link_radius}"/>
+	    </geometry>
+	</collision>
+    <xacro:inertia_wheel />
+</link>
+<!--######################################################### -->
 <joint name="wheel6_joint" type="continuous">
 	<parent link="body_link"/>
 	<child link="wheel6_link"/>
-	<origin xyz="1.0 0.4 -0.5" rpy="0 0 0"/>
+	<origin xyz="0 ${body_link_y_dim/2+wheel_link_length/2} ${wheel_link_z_location}" rpy="0 0 0"/>
 	<axis xyz="0 1 0"/>
 	<limit effort="1000" velocity="1000"/>
@@ -185,17 +184,17 @@
 </joint>
 <link name="wheel6_link">
-	<visual>
-		<origin rpy="1.570795 0 0" xyz="0 0 0"/>
-		<geometry>
-			<cylinder length="${wheel_link_length}" radius="${wheel_link_radius}"/>
-		</geometry>
-	</visual>
-	<collision>
-		<origin rpy="1.570795 0 0" xyz="0 0 0"/>
-		<geometry>
-			<cylinder length="${wheel_link_length}" radius="${wheel_link_radius}"/>
-		</geometry>
-	</collision>
-	<xacro:inertia_wheel />
+    <visual>
+	    <origin rpy="1.570795 0 0" xyz="0 0 0"/>
+	    <geometry>
+	        <cylinder length="${wheel_link_length}" radius="${wheel_link_radius}"/>
+	    </geometry>
+	</visual>
+	<collision>
+	    <origin rpy="1.570795 0 0" xyz="0 0 0"/>
+	    <geometry>
+	        <cylinder length="${wheel_link_length}" radius="${wheel_link_radius}"/>
+	    </geometry>
+	</collision>
+    <xacro:inertia_wheel />
 </link>
 </robot>
